File: Snake_3D_KiCAD/Snake_3D_KiCAD.kicad_sch (KiCad schematic)
At the start: 8 parts, among them J1 Conn_01x08, J2 Conn_01x08, J3 top LED pannel, J4 lateral led pannels, J5 Score Display 1, J6 Score Display 2, J7 Joystick

Commit message: continued working on pcb
Parts:
- removed J1, J2: Conn_01x08, symbol Connector_Generic:Conn_01x08
- added A3: Pololu_Breakout_DRV8825, Module:Pololu_Breakout-16_15.2x20.3mm, symbol Driver_Motor:Pololu_Breakout_DRV8825
- added J1: Conn_01x02_Pin, Connector_JST:JST_GH_SM02B-GHS-TB_1x02-1MP_P1.25mm_Horizontal, symbol Connector:Conn_01x02_Pin
- added J9: stepper motor pins, Connector_PinHeader_2.54mm:PinHeader_1x04_P2.54mm_Vertical, symbol Connector:Conn_01x04_Pin
- added U2: MAX98357A, Package_DFN_QFN:TQFN-16-1EP_3x3mm_P0.5mm_EP1.23x1.23mm, symbol Audio:MAX98357A
- J3, J4: footprint (none) -> Connector_PinHeader_2.54mm:PinHeader_1x03_P2.54mm_Vertical
- J5, J6: footprint (none) -> Connector_PinHeader_2.54mm:PinHeader_1x04_P2.54mm_Vertical
- J7: footprint (none) -> Connector_PinHeader_2.54mm:PinHeader_1x05_P2.54mm_Vertical
Connections:
- net +3.3V: now also U2.7 (VDD), U2.8 (VDD)
- net GND: now also A3.1 (GND), A3.7 (GND), U2.11 (GND), U2.15 (GND), U2.3 (GND), U2.4 (~{SD_MODE})
- net at A1.10 (GPIO7): now also A3.9 (~{EN})
- net at A1.11 (GPIO8): now also A3.15 (STEP)
- net at A1.12 (GPIO9): now also U2.16 (BCLK)
- net at A1.14 (GPIO10): now also U2.14 (LRCLK)
- net at A1.15 (GPIO11): now also U2.1 (DIN)
- net at A1.4 (GPIO2): now also A3.16 (DIR)
- net at A1.6 (GPIO4): now also A3.14 (~{SLP})
- net at A1.7 (GPIO5): now also A3.13 (~{RST})
- net at A1.9 (GPIO6): now also A3.2 (~{FLT})
- new net: A3.4 (A1), J9.A1
- new net: A3.3 (A2), J9.A2
- new net: A3.5 (B1), J9.B1
- new net: A3.6 (B2), J9.B2
- new net: J1.1 (Pin_1), U2.10 (OUTN)
- new net: J1.2 (Pin_2), U2.9 (OUTP)
- no-connect marks 0 -> 5

Commit message: finished pcb design
Parts:
- removed J1: Conn_01x02_Pin, Connector_JST:JST_GH_SM02B-GHS-TB_1x02-1MP_P1.25mm_Horizontal, symbol Connector:Conn_01x02_Pin
- removed U2: MAX98357A, Package_DFN_QFN:TQFN-16-1EP_3x3mm_P0.5mm_EP1.23x1.23mm, symbol Audio:MAX98357A
- added J2: Conn_01x07, Connector_PinHeader_2.54mm:PinHeader_1x07_P2.54mm_Vertical, symbol Connector_Generic:Conn_01x07
Connections:
- net +3V3 is gone; now on net +3.3V: A1.36 (3V3)
- net +3.3V: now also J5.3 (VCC), J6.3 (VCC), J2.7 (Pin_7); no longer J5.VCC, J6.VCC
- net +5V: now also J3.1 (VIN), J4.1 (VIN), J7.2 (+5V); no longer J3.VIN, J4.VIN, J7.+5V
- net GND: now also J3.3 (GND), J4.3 (GND), J5.4 (GND), J6.4 (GND), J7.1 (GND), J2.5 (Pin_5), J2.6 (Pin_6); no longer J3.GND, J4.GND, J5.GND, J6.GND, J7.GND
- net at A3.4 (A1): now also J9.4 (A1); no longer J9.A1
- net at A3.3 (A2): now also J9.3 (A2); no longer J9.A2
- net at A3.5 (B1): now also J9.2 (B1); no longer J9.B1
- net at A3.6 (B2): now also J9.1 (B2); no longer J9.B2
- net at A1.5 (GPIO3): now also J3.2 (DIN_0); no longer J3.DIN_0
- net at A1.1 (GPIO0): now also J4.2 (DIN_0); no longer J4.DIN_0
- net at A1.12 (GPIO9): now also J2.2 (Pin_2)
- net at A1.14 (GPIO10): now also J2.1 (Pin_1)
- net at A1.15 (GPIO11): now also J2.3 (Pin_3)
- net at A1.25 (GPIO19): now also J7.5 (SW); no longer J7.SW
- net at A1.26 (GPIO20): now also J6.1 (CLK); no longer J6.CLK
- net at A1.27 (GPIO21): now also J6.2 (DIO); no longer J6.DIO
- net at A1.29 (GPIO22): now also J5.1 (CLK); no longer J5.CLK
- net at A1.31 (GPIO26_ADC0): now also J7.3 (VRX); no longer J7.VRX
- net at A1.32 (GPIO27_ADC1): now also J7.4 (VRY); no longer J7.VRY
- net at A1.34 (GPIO28_ADC2): now also J5.2 (DIO); no longer J5.DIO
- no-connect marks 5 -> 18
Other:
- moved on the sheet: J3, J4, J9
